File: ALU/kicad/1BitALU/1BitALU.sch (KiCad schematic (older format))
At the start: 21 parts, among them P1 CONN_6, P2 CONN_2, P3 Power

Commit message: more updates
Parts:
- D1, D2, D3, D4, D5, D6, D7, D8, D9: footprint ~ -> custom:90LED
- P1: footprint (none) -> Socket_Strips:Socket_Strip_Angled_1x06
- P2, P3: footprint (none) -> Socket_Strips:Socket_Strip_Angled_1x02
- R1, R2, R3, R4, R5, R6, R7, R8, R9: footprint ~ -> Discret:R4
Changed lines of the file:
@@
 $EndComp
 Wire Wire Line
-	1850 5600 3400 5600
+	2650 5600 3400 5600
 Wire Wire Line
 	2700 6200 3400 6200
@@
 F 0 "D1" H 4450 4750 50  0000 C CNN
 F 1 "LED" H 4450 4550 50  0000 C CNN
-F 2 "~" H 4450 4650 60  0000 C CNN
+F 2 "custom:90LED" H 4450 4650 60  0000 C CNN
 F 3 "~" H 4450 4650 60  0000 C CNN
 	1    4450 4650
@@
 F 0 "D2" H 4450 5100 50  0000 C CNN
 F 1 "LED" H 4450 4900 50  0000 C CNN
-F 2 "~" H 4450 5000 60  0000 C CNN
+F 2 "custom:90LED" H 4450 5000 60  0000 C CNN
 F 3 "~" H 4450 5000 60  0000 C CNN
 	1    4450 5000
@@
 F 0 "D3" H 4450 5400 50  0000 C CNN
 F 1 "LED" H 4450 5200 50  0000 C CNN
-F 2 "~" H 4450 5300 60  0000 C CNN
+F 2 "custom:90LED" H 4450 5300 60  0000 C CNN
 F 3 "~" H 4450 5300 60  0000 C CNN
 	1    4450 5300
@@
 F 0 "D4" H 4450 5700 50  0000 C CNN
 F 1 "LED" H 4450 5500 50  0000 C CNN
-F 2 "~" H 4450 5600 60  0000 C CNN
+F 2 "custom:90LED" H 4450 5600 60  0000 C CNN
 F 3 "~" H 4450 5600 60  0000 C CNN
 	1    4450 5600
@@
 F 0 "D5" H 4450 6000 50  0000 C CNN
 F 1 "LED" H 4450 5800 50  0000 C CNN
-F 2 "~" H 4450 5900 60  0000 C CNN
+F 2 "custom:90LED" H 4450 5900 60  0000 C CNN
 F 3 "~" H 4450 5900 60  0000 C CNN
 	1    4450 5900
@@
 F 0 "D6" H 4450 6300 50  0000 C CNN
 F 1 "LED" H 4450 6100 50  0000 C CNN
-F 2 "~" H 4450 6200 60  0000 C CNN
+F 2 "custom:90LED" H 4450 6200 60  0000 C CNN
 F 3 "~" H 4450 6200 60  0000 C CNN
 	1    4450 6200
@@
 F 0 "D7" H 4450 6650 50  0000 C CNN
 F 1 "LED" H 4450 6450 50  0000 C CNN
-F 2 "~" H 4450 6550 60  0000 C CNN
+F 2 "custom:90LED" H 4450 6550 60  0000 C CNN
 F 3 "~" H 4450 6550 60  0000 C CNN
 	1    4450 6550
@@
 F 0 "D8" H 4450 7000 50  0000 C CNN
 F 1 "LED" H 4450 6800 50  0000 C CNN
-F 2 "~" H 4450 6900 60  0000 C CNN
+F 2 "custom:90LED" H 4450 6900 60  0000 C CNN
 F 3 "~" H 4450 6900 60  0000 C CNN
 	1    4450 6900
@@
 $EndComp
 Wire Wire Line
-	4650 6900 4950 6900
+	4650 6900 4800 6900
+Wire Wire Line
+	4800 6900 4950 6900
 Wire Wire Line
 	4950 6900 4950 7000
@@
 	4650 4650 4800 4700
 Wire Wire Line
-	4800 4700 4800 6900
+	4800 4700 4800 5000
+Wire Wire Line
+	4800 5000 4800 5300
+Wire Wire Line
+	4800 5300 4800 5600
+Wire Wire Line
+	4800 5600 4800 5900
+Wire Wire Line
+	4800 5900 4800 6200
+Wire Wire Line
+	4800 6200 4800 6550
+Wire Wire Line
+	4800 6550 4800 6900
 Wire Wire Line
 	4800 5000 4650 5000
@@
 F 0 "R1" V 3730 4650 40  0000 C CNN
 F 1 "100 Ohm" V 3657 4651 40  0000 C CNN
-F 2 "~" V 3580 4650 30  0000 C CNN
+F 2 "Discret:R4" V 3580 4650 30  0000 C CNN
 F 3 "~" H 3650 4650 30  0000 C CNN
 	1    3650 4650
@@
 F 0 "R2" V 3730 5000 40  0000 C CNN
 F 1 "100 Ohm" V 3657 5001 40  0000 C CNN
-F 2 "~" V 3580 5000 30  0000 C CNN
+F 2 "Discret:R4" V 3580 5000 30  0000 C CNN
 F 3 "~" H 3650 5000 30  0000 C CNN
 	1    3650 5000
@@
 F 0 "R4" V 3730 5600 40  0000 C CNN
 F 1 "100 Ohm" V 3657 5601 40  0000 C CNN
-F 2 "~" V 3580 5600 30  0000 C CNN
+F 2 "Discret:R4" V 3580 5600 30  0000 C CNN
 F 3 "~" H 3650 5600 30  0000 C CNN
 	1    3650 5600
@@
 F 0 "R3" V 3730 5300 40  0000 C CNN
 F 1 "100 Ohm" V 3657 5301 40  0000 C CNN
-F 2 "~" V 3580 5300 30  0000 C CNN
+F 2 "Discret:R4" V 3580 5300 30  0000 C CNN
 F 3 "~" H 3650 5300 30  0000 C CNN
 	1    3650 5300
@@
 F 0 "R5" V 3730 5900 40  0000 C CNN
 F 1 "100 Ohm" V 3657 5901 40  0000 C CNN
-F 2 "~" V 3580 5900 30  0000 C CNN
+F 2 "Discret:R4" V 3580 5900 30  0000 C CNN
 F 3 "~" H 3650 5900 30  0000 C CNN
 	1    3650 5900
@@
 F 0 "R6" V 3730 6200 40  0000 C CNN
 F 1 "100 Ohm" V 3657 6201 40  0000 C CNN
-F 2 "~" V 3580 6200 30  0000 C CNN
+F 2 "Discret:R4" V 3580 6200 30  0000 C CNN
 F 3 "~" H 3650 6200 30  0000 C CNN
 	1    3650 6200
@@
 F 0 "R7" V 3730 6550 40  0000 C CNN
 F 1 "100 Ohm" V 3657 6551 40  0000 C CNN
-F 2 "~" V 3580 6550 30  0000 C CNN
+F 2 "Discret:R4" V 3580 6550 30  0000 C CNN
 F 3 "~" H 3650 6550 30  0000 C CNN
 	1    3650 6550
@@
 F 0 "R8" V 3730 6900 40  0000 C CNN
 F 1 "100 Ohm" V 3657 6901 40  0000 C CNN
-F 2 "~" V 3580 6900 30  0000 C CNN
+F 2 "Discret:R4" V 3580 6900 30  0000 C CNN
 F 3 "~" H 3650 6900 30  0000 C CNN
 	1    3650 6900
@@
 F 0 "P1" V 7250 4500 60  0000 C CNN
 F 1 "CONN_6" V 7350 4500 60  0000 C CNN
-F 2 "" H 7300 4500 60  0000 C CNN
+F 2 "Socket_Strips:Socket_Strip_Angled_1x06" H 7300 4500 60  0001 C CNN
 F 3 "" H 7300 4500 60  0000 C CNN
 	1    7300 4500
@@
 F 0 "P2" V 7350 6250 40  0000 C CNN
 F 1 "CONN_2" V 7450 6250 40  0000 C CNN
-F 2 "" H 7400 6250 60  0000 C CNN
+F 2 "Socket_Strips:Socket_Strip_Angled_1x02" H 7400 6250 60  0001 C CNN
 F 3 "" H 7400 6250 60  0000 C CNN
 	1    7400 6250
@@
 F 0 "D9" H 8850 4400 50  0000 C CNN
 F 1 "LED" H 8850 4200 50  0000 C CNN
-F 2 "~" H 8850 4300 60  0000 C CNN
+F 2 "custom:90LED" H 8850 4300 60  0000 C CNN
 F 3 "~" H 8850 4300 60  0000 C CNN
 	1    8850 4300
@@
 F 0 "R9" V 8730 4550 40  0000 C CNN
 F 1 "100 Ohm" V 8657 4551 40  0000 C CNN
-F 2 "~" V 8580 4550 30  0000 C CNN
+F 2 "Discret:R4" V 8580 4550 30  0000 C CNN
 F 3 "~" H 8650 4550 30  0000 C CNN
 	1    8650 4550
@@
 F 0 "P3" V 8850 6250 40  0000 C CNN
 F 1 "Power" V 8950 6250 40  0000 C CNN
-F 2 "" H 8900 6250 60  0000 C CNN
+F 2 "Socket_Strips:Socket_Strip_Angled_1x02" H 8900 6250 60  0001 C CNN
 F 3 "" H 8900 6250 60  0000 C CNN
 	1    8900 6250
@@
 Wire Wire Line
 	6750 5050 6950 4750
-Text GLabel 1850 5600 0    60   Input ~ 0
+Text GLabel 2650 5600 0    60   Input ~ 0
 A
 Text GLabel 6250 4650 0    60   Input ~ 0
