File: ALU/kicad/1BitALU/sectionA.sch (KiCad schematic (older format))
At the start: 7 parts, among them U10 and3a, U11 or2a, U12 and3b, U13 inv3b, U14 and3c, U15 or3a, U9 or2b

Commit message: * improvements
Changed lines of the file:
@@
 LIBS:valves
 LIBS:1BitALU-cache
-EELAYER 27 0
+EELAYER 25 0
 EELAYER END
 $Descr USLetter 11000 8500
@@
 Sheet 2 6
 Title "Relay Computer - 1 Bit ALU"
-Date "8 mar 2015"
-Rev "1.5"
-Comp "Vincent Fumo"
-Comment1 ""
+Date "Tuesday, March 10, 2015"
+Rev "1.6"
+Comp "http://vfumo.info"
+Comment1 "Vincent E. Fumo II"
 Comment2 ""
 Comment3 ""
@@
 L GND #PWR07
 U 1 1 54D012DC
-P 4450 3400
-F 0 "#PWR07" H 4450 3400 30  0001 C CNN
-F 1 "GND" H 4450 3330 30  0001 C CNN
-F 2 "" H 4450 3400 60  0000 C CNN
-F 3 "" H 4450 3400 60  0000 C CNN
-	1    4450 3400
+P 4100 3300
+F 0 "#PWR07" H 4100 3300 30  0001 C CNN
+F 1 "GND" H 4100 3230 30  0001 C CNN
+F 2 "" H 4100 3300 60  0000 C CNN
+F 3 "" H 4100 3300 60  0000 C CNN
+	1    4100 3300
 	1    0    0    -1
 $EndComp
@@
 	1800 3400 1800 3500
 Wire Wire Line
-	4100 3100 4450 3400
+	4100 3100 4100 3300
 $Comp
 L +5V #PWR08
@@
 L +5V #PWR011
 U 1 1 54D016DF
-P 7850 2200
-F 0 "#PWR011" H 7850 2290 20  0001 C CNN
-F 1 "+5V" H 7850 2290 30  0000 C CNN
-F 2 "" H 7850 2200 60  0000 C CNN
-F 3 "" H 7850 2200 60  0000 C CNN
-	1    7850 2200
+P 7900 2600
+F 0 "#PWR011" H 7900 2690 20  0001 C CNN
+F 1 "+5V" H 7900 2690 30  0000 C CNN
+F 2 "" H 7900 2600 60  0000 C CNN
+F 3 "" H 7900 2600 60  0000 C CNN
+	1    7900 2600
 	1    0    0    -1
 $EndComp
@@
 Wire Wire Line
 	9100 5600 9100 5500
-Wire Wire Line
-	7850 2200 7850 2250
-Wire Wire Line
-	7850 2250 7750 2650
 Wire Wire Line
 	5150 3600 5850 3600
@@
 Text GLabel 2100 1800 2    60   Input ~ 0
 B Actual
+Wire Wire Line
+	7750 2650 7900 2650
+Wire Wire Line
+	7900 2650 7900 2600
 $EndSCHEMATC

Commit message: more updates
Parts:
- U10, U11, U12, U14, U15, U9: footprint (none) -> custom:211ARelay
- U13: footprint FBR211A -> custom:211ARelay
Changed lines of the file:
@@
 F 0 "U9" H 2150 2200 60  0000 C CNN
 F 1 "or2b" H 1800 2700 60  0000 C CNN
-F 2 "" H 800 2650 60  0000 C CNN
+F 2 "custom:211ARelay" H 800 2650 60  0001 C CNN
 F 3 "" H 800 2650 60  0000 C CNN
 	1    1800 2700
@@
 F 0 "U11" H 4450 1900 60  0000 C CNN
 F 1 "or2a" H 4100 2400 60  0000 C CNN
-F 2 "" H 3100 2350 60  0000 C CNN
+F 2 "custom:211ARelay" H 3100 2350 60  0001 C CNN
 F 3 "" H 3100 2350 60  0000 C CNN
 	1    4100 2400
@@
 F 0 "U10" H 3400 3800 60  0000 C CNN
 F 1 "and3a" H 3050 4300 60  0000 C CNN
-F 2 "" H 2050 4250 60  0000 C CNN
+F 2 "custom:211ARelay" H 2050 4250 60  0001 C CNN
 F 3 "" H 2050 4250 60  0000 C CNN
 	1    3050 4300
@@
 F 0 "U12" H 5500 3800 60  0000 C CNN
 F 1 "and3b" H 5150 4300 60  0000 C CNN
-F 2 "" H 4150 4250 60  0000 C CNN
+F 2 "custom:211ARelay" H 4150 4250 60  0001 C CNN
 F 3 "" H 4150 4250 60  0000 C CNN
 	1    5150 4300
@@
 F 0 "U15" H 9450 4300 60  0000 C CNN
 F 1 "or3a" H 9100 4800 60  0000 C CNN
-F 2 "" H 8100 4750 60  0000 C CNN
+F 2 "custom:211ARelay" H 8100 4750 60  0001 C CNN
 F 3 "" H 8100 4750 60  0000 C CNN
 	1    9100 4800
@@
 F 0 "U14" H 7500 3800 60  0000 C CNN
 F 1 "and3c" H 7150 4300 60  0000 C CNN
-F 2 "" H 6150 4250 60  0000 C CNN
+F 2 "custom:211ARelay" H 6150 4250 60  0001 C CNN
 F 3 "" H 6150 4250 60  0000 C CNN
 	1    7150 4300
@@
 F 0 "U13" H 7400 1950 60  0000 C CNN
 F 1 "inv3b" H 7050 2450 60  0000 C CNN
-F 2 "FBR211A" H 6600 1950 60  0000 C CNN
+F 2 "custom:211ARelay" H 6600 1950 60  0000 C CNN
 F 3 "" H 6050 2400 60  0000 C CNN
 	1    7050 2450
