File: ALU/kicad/1BitALU/sectionB.sch (KiCad schematic (older format))
At the start: 8 parts, among them U1 xor3a, U2 and2a, U3 xor3b, U4 and2b, U5 or1b, U6 and1a, U7 and1b, U8 or1a

Commit message: * improvements
Other:
- moved on the sheet: U2
Changed lines of the file:
@@
 LIBS:valves
 LIBS:1BitALU-cache
-EELAYER 27 0
+EELAYER 25 0
 EELAYER END
 $Descr USLetter 11000 8500
 encoding utf-8
 Sheet 6 6
-Title ""
-Date "8 mar 2015"
-Rev ""
-Comp ""
-Comment1 ""
+Title "Relay Computer - 1 Bit ALU"
+Date "Tuesday, March 10, 2015"
+Rev "1.6"
+Comp "http://vfumo.info"
+Comment1 "Vincent E. Fumo II"
 Comment2 ""
 Comment3 ""
@@
 L FBR211 U2
 U 1 1 54D2A2C2
-P 2350 4300
-F 0 "U2" H 2700 3800 60  0000 C CNN
-F 1 "and2a" H 2350 4300 60  0000 C CNN
-F 2 "~" H 1350 4250 60  0000 C CNN
-F 3 "~" H 1350 4250 60  0000 C CNN
-	1    2350 4300
+P 2300 4700
+F 0 "U2" H 2650 4200 60  0000 C CNN
+F 1 "and2a" H 2300 4700 60  0000 C CNN
+F 2 "~" H 1300 4650 60  0000 C CNN
+F 3 "~" H 1300 4650 60  0000 C CNN
+	1    2300 4700
 	-1   0    0    -1
 $EndComp
@@
 L GND #PWR050
 U 1 1 54D2A4FF
-P 2350 5150
-F 0 "#PWR050" H 2350 5150 30  0001 C CNN
-F 1 "GND" H 2350 5080 30  0001 C CNN
-F 2 "" H 2350 5150 60  0000 C CNN
-F 3 "" H 2350 5150 60  0000 C CNN
-	1    2350 5150
+P 2300 5500
+F 0 "#PWR050" H 2300 5500 30  0001 C CNN
+F 1 "GND" H 2300 5430 30  0001 C CNN
+F 2 "" H 2300 5500 60  0000 C CNN
+F 3 "" H 2300 5500 60  0000 C CNN
+	1    2300 5500
 	1    0    0    -1
 $EndComp
@@
 L +5V #PWR056
 U 1 1 54D2A5B4
-P 1500 4100
-F 0 "#PWR056" H 1500 4190 20  0001 C CNN
-F 1 "+5V" H 1500 4190 30  0000 C CNN
-F 2 "" H 1500 4100 60  0000 C CNN
-F 3 "" H 1500 4100 60  0000 C CNN
-	1    1500 4100
+P 1450 4500
+F 0 "#PWR056" H 1450 4590 20  0001 C CNN
+F 1 "+5V" H 1450 4590 30  0000 C CNN
+F 2 "" H 1450 4500 60  0000 C CNN
+F 3 "" H 1450 4500 60  0000 C CNN
+	1    1450 4500
 	1    0    0    -1
 $EndComp
@@
 L +5V #PWR057
 U 1 1 54D2A5CD
-P 1400 1550
-F 0 "#PWR057" H 1400 1640 20  0001 C CNN
-F 1 "+5V" H 1400 1640 30  0000 C CNN
-F 2 "" H 1400 1550 60  0000 C CNN
-F 3 "" H 1400 1550 60  0000 C CNN
-	1    1400 1550
+P 1350 1950
+F 0 "#PWR057" H 1350 2040 20  0001 C CNN
+F 1 "+5V" H 1350 2040 30  0000 C CNN
+F 2 "" H 1350 1950 60  0000 C CNN
+F 3 "" H 1350 1950 60  0000 C CNN
+	1    1350 1950
 	1    0    0    -1
 $EndComp
@@
 L +5V #PWR058
 U 1 1 54D2A5FD
-P 5450 2550
-F 0 "#PWR058" H 5450 2640 20  0001 C CNN
-F 1 "+5V" H 5450 2640 30  0000 C CNN
-F 2 "" H 5450 2550 60  0000 C CNN
-F 3 "" H 5450 2550 60  0000 C CNN
-	1    5450 2550
+P 5450 2950
+F 0 "#PWR058" H 5450 3040 20  0001 C CNN
+F 1 "+5V" H 5450 3040 30  0000 C CNN
+F 2 "" H 5450 2950 60  0000 C CNN
+F 3 "" H 5450 2950 60  0000 C CNN
+	1    5450 2950
 	1    0    0    -1
 $EndComp
@@
 L +5V #PWR059
 U 1 1 54D2A611
-P 5350 5300
-F 0 "#PWR059" H 5350 5390 20  0001 C CNN
-F 1 "+5V" H 5350 5390 30  0000 C CNN
-F 2 "" H 5350 5300 60  0000 C CNN
-F 3 "" H 5350 5300 60  0000 C CNN
-	1    5350 5300
+P 5350 5700
+F 0 "#PWR059" H 5350 5790 20  0001 C CNN
+F 1 "+5V" H 5350 5790 30  0000 C CNN
+F 2 "" H 5350 5700 60  0000 C CNN
+F 3 "" H 5350 5700 60  0000 C CNN
+	1    5350 5700
 	1    0    0    -1
 $EndComp
@@
 L +5V #PWR060
 U 1 1 54D2A625
-P 8200 4150
-F 0 "#PWR060" H 8200 4240 20  0001 C CNN
-F 1 "+5V" H 8200 4240 30  0000 C CNN
-F 2 "" H 8200 4150 60  0000 C CNN
-F 3 "" H 8200 4150 60  0000 C CNN
-	1    8200 4150
+P 8200 4550
+F 0 "#PWR060" H 8200 4640 20  0001 C CNN
+F 1 "+5V" H 8200 4640 30  0000 C CNN
+F 2 "" H 8200 4550 60  0000 C CNN
+F 3 "" H 8200 4550 60  0000 C CNN
+	1    8200 4550
 	1    0    0    -1
 $EndComp
@@
 	2950 1950 3400 1550
 Wire Wire Line
-	4150 4500 3100 4100
+	4150 4500 3050 4500
 Wire Wire Line
 	5600 4100 6150 4800
@@
 	4850 5000 4850 5150
 Wire Wire Line
-	2350 5000 2350 5150
+	2300 5400 2300 5500
 Wire Wire Line
 	2200 2450 2200 2600
@@
 	9050 5050 9050 5250
 Wire Wire Line
-	1500 1950 1400 1550
-Wire Wire Line
-	1650 4100 1500 4100
-Wire Wire Line
-	8350 4550 8200 4150
-Wire Wire Line
-	5450 2550 5650 2950
-Wire Wire Line
-	5350 5300 5450 5700
+	1500 1950 1350 1950
+Wire Wire Line
+	1600 4500 1450 4500
+Wire Wire Line
+	8350 4550 8200 4550
+Wire Wire Line
+	5450 2950 5650 2950
+Wire Wire Line
+	5350 5700 5450 5700
 Wire Wire Line
 	2400 1050 2200 1050
@@
 	4850 1550 5100 1550
 Wire Wire Line
-	2550 3600 2350 3600
+	2650 4000 2300 4000
 Wire Wire Line
 	5600 4100 6100 4100
@@
 Text GLabel 6100 4100 2    60   Input ~ 0
 AND Out
-Text GLabel 2550 3600 2    60   Input ~ 0
+Text GLabel 2650 4000 2    60   Input ~ 0
 A
 Text GLabel 6700 2050 2    60   Input ~ 0
@@
 Text GLabel 5100 1550 2    60   Input ~ 0
 B Actual
-Text GLabel 5150 3500 2    60   Input ~ 0
+Text GLabel 5150 3600 2    60   Input ~ 0
 B Actual
 Wire Wire Line
-	4850 3600 5150 3500
+	4850 3600 5150 3600
 $EndSCHEMATC

Commit message: more updates
Parts:
- U1, U2, U3, U4, U5, U6, U7, U8: footprint ~ -> custom:211ARelay
Changed lines of the file:
@@
 F 0 "U1" H 2550 1250 60  0000 C CNN
 F 1 "xor3a" H 2200 1750 60  0000 C CNN
-F 2 "~" H 1200 1700 60  0000 C CNN
+F 2 "custom:211ARelay" H 1200 1700 60  0000 C CNN
 F 3 "~" H 1200 1700 60  0000 C CNN
 	1    2200 1750
@@
 F 0 "U2" H 2650 4200 60  0000 C CNN
 F 1 "and2a" H 2300 4700 60  0000 C CNN
-F 2 "~" H 1300 4650 60  0000 C CNN
+F 2 "custom:211ARelay" H 1300 4650 60  0000 C CNN
 F 3 "~" H 1300 4650 60  0000 C CNN
 	1    2300 4700
@@
 F 0 "U4" H 5200 3800 60  0000 C CNN
 F 1 "and2b" H 4850 4300 60  0000 C CNN
-F 2 "~" H 3850 4250 60  0000 C CNN
+F 2 "custom:211ARelay" H 3850 4250 60  0000 C CNN
 F 3 "~" H 3850 4250 60  0000 C CNN
 	1    4850 4300
@@
 F 0 "U6" H 6700 2250 60  0000 C CNN
 F 1 "and1a" H 6350 2750 60  0000 C CNN
-F 2 "~" H 5350 2700 60  0000 C CNN
+F 2 "custom:211ARelay" H 5350 2700 60  0000 C CNN
 F 3 "~" H 5350 2700 60  0000 C CNN
 	1    6350 2750
@@
 F 0 "U5" H 6500 5000 60  0000 C CNN
 F 1 "or1b" H 6150 5500 60  0000 C CNN
-F 2 "~" H 5150 5450 60  0000 C CNN
+F 2 "custom:211ARelay" H 5150 5450 60  0000 C CNN
 F 3 "~" H 5150 5450 60  0000 C CNN
 	1    6150 5500
@@
 F 0 "U8" H 9400 3850 60  0000 C CNN
 F 1 "or1a" H 9050 4350 60  0000 C CNN
-F 2 "~" H 8050 4300 60  0000 C CNN
+F 2 "custom:211ARelay" H 8050 4300 60  0000 C CNN
 F 3 "~" H 8050 4300 60  0000 C CNN
 	1    9050 4350
@@
 F 0 "U7" H 8450 2250 60  0000 C CNN
 F 1 "and1b" H 8100 2750 60  0000 C CNN
-F 2 "~" H 7100 2700 60  0000 C CNN
+F 2 "custom:211ARelay" H 7100 2700 60  0000 C CNN
 F 3 "~" H 7100 2700 60  0000 C CNN
 	1    8100 2750
@@
 F 0 "U3" H 4500 1250 60  0000 C CNN
 F 1 "xor3b" H 4150 1750 60  0000 C CNN
-F 2 "~" H 3150 1700 60  0000 C CNN
+F 2 "custom:211ARelay" H 3150 1700 60  0000 C CNN
 F 3 "~" H 3150 1700 60  0000 C CNN
 	1    4150 1750
