File: ALU/kicad/1BitALU/sectionC.sch (KiCad schematic (older format))
At the start: 8 parts, among them U16 xor1b, U17 xor1a, U18 xor2b, U19 and4a, U20 xor2a, U21 and4b, U22 and4c, U23 or3b

Commit message: * improvements
Other:
- moved on the sheet: U18, U19, U20, U21, U22, U23

Commit message: more updates
Parts:
- U16, U17, U18, U19, U20, U21, U22, U23: footprint ~ -> custom:211ARelay
Changed lines of the file:
@@
 F 0 "U16" H 2000 1150 60  0000 C CNN
 F 1 "xor1b" H 1650 1650 60  0000 C CNN
-F 2 "~" H 650 1600 60  0000 C CNN
+F 2 "custom:211ARelay" H 650 1600 60  0000 C CNN
 F 3 "~" H 650 1600 60  0000 C CNN
 	1    1650 1650
@@
 F 0 "U17" H 3850 1150 60  0000 C CNN
 F 1 "xor1a" H 3500 1650 60  0000 C CNN
-F 2 "~" H 2500 1600 60  0000 C CNN
+F 2 "custom:211ARelay" H 2500 1600 60  0000 C CNN
 F 3 "~" H 2500 1600 60  0000 C CNN
 	1    3500 1650
@@
 F 0 "U19" H 5200 2850 60  0000 C CNN
 F 1 "and4a" H 4850 3350 60  0000 C CNN
-F 2 "~" H 3850 3300 60  0000 C CNN
+F 2 "custom:211ARelay" H 3850 3300 60  0000 C CNN
 F 3 "~" H 3850 3300 60  0000 C CNN
 	1    4850 3350
@@
 F 0 "U23" H 9750 4200 60  0000 C CNN
 F 1 "or3b" H 9400 4700 60  0000 C CNN
-F 2 "~" H 8400 4650 60  0000 C CNN
+F 2 "custom:211ARelay" H 8400 4650 60  0000 C CNN
 F 3 "~" H 8400 4650 60  0000 C CNN
 	1    9400 4700
@@
 F 0 "U18" H 2750 5050 60  0000 C CNN
 F 1 "xor2b" H 2400 5550 60  0000 C CNN
-F 2 "~" H 1400 5500 60  0000 C CNN
+F 2 "custom:211ARelay" H 1400 5500 60  0000 C CNN
 F 3 "~" H 1400 5500 60  0000 C CNN
 	1    2400 5550
@@
 F 0 "U20" H 4550 5050 60  0000 C CNN
 F 1 "xor2a" H 4200 5550 60  0000 C CNN
-F 2 "~" H 3200 5500 60  0000 C CNN
+F 2 "custom:211ARelay" H 3200 5500 60  0000 C CNN
 F 3 "~" H 3200 5500 60  0000 C CNN
 	1    4200 5550
@@
 F 0 "U22" H 8650 2850 60  0000 C CNN
 F 1 "and4c" H 8300 3350 60  0000 C CNN
-F 2 "~" H 7300 3300 60  0000 C CNN
+F 2 "custom:211ARelay" H 7300 3300 60  0000 C CNN
 F 3 "~" H 7300 3300 60  0000 C CNN
 	1    8300 3350
@@
 F 0 "U21" H 6900 2850 60  0000 C CNN
 F 1 "and4b" H 6550 3350 60  0000 C CNN
-F 2 "~" H 5550 3300 60  0000 C CNN
+F 2 "custom:211ARelay" H 5550 3300 60  0000 C CNN
 F 3 "~" H 5550 3300 60  0000 C CNN
 	1    6550 3350
