File: ALU/kicad/1BitALU/sectionD.sch (KiCad schematic (older format))
At the start: 5 parts, among them U24 and5a, U25 and5b, U26 inv5c, U27 and5c, U28 or3c

Commit message: * improvements
Other:
- moved on the sheet: U26
Changed lines of the file:
@@
 LIBS:valves
 LIBS:1BitALU-cache
-EELAYER 27 0
+EELAYER 25 0
 EELAYER END
 $Descr USLetter 11000 8500
 encoding utf-8
 Sheet 4 6
-Title ""
-Date "8 mar 2015"
-Rev ""
-Comp ""
-Comment1 ""
+Title "Relay Computer - 1 Bit ALU"
+Date "Tuesday, March 10, 2015"
+Rev "1.6"
+Comp "http://vfumo.info"
+Comment1 "Vincent E. Fumo II"
 Comment2 ""
 Comment3 ""
@@
 	5900 3400 5900 2100
 Wire Wire Line
-	5900 2100 5650 2300
+	5900 2100 5650 2100
 $Comp
 L +5V #PWR030
 U 1 1 54D2DC83
-P 4200 1700
-F 0 "#PWR030" H 4200 1790 20  0001 C CNN
-F 1 "+5V" H 4200 1790 30  0000 C CNN
-F 2 "" H 4200 1700 60  0000 C CNN
-F 3 "" H 4200 1700 60  0000 C CNN
-	1    4200 1700
+P 4050 1700
+F 0 "#PWR030" H 4050 1790 20  0001 C CNN
+F 1 "+5V" H 4050 1790 30  0000 C CNN
+F 2 "" H 4050 1700 60  0000 C CNN
+F 3 "" H 4050 1700 60  0000 C CNN
+	1    4050 1700
 	1    0    0    -1
 $EndComp
@@
 L +5V #PWR031
 U 1 1 54D2DC92
-P 1300 3850
-F 0 "#PWR031" H 1300 3940 20  0001 C CNN
-F 1 "+5V" H 1300 3940 30  0000 C CNN
-F 2 "" H 1300 3850 60  0000 C CNN
-F 3 "" H 1300 3850 60  0000 C CNN
-	1    1300 3850
+P 1300 4300
+F 0 "#PWR031" H 1300 4390 20  0001 C CNN
+F 1 "+5V" H 1300 4390 30  0000 C CNN
+F 2 "" H 1300 4300 60  0000 C CNN
+F 3 "" H 1300 4300 60  0000 C CNN
+	1    1300 4300
 	1    0    0    -1
 $EndComp
@@
 L +5V #PWR032
 U 1 1 54D2DCA1
-P 9000 4650
-F 0 "#PWR032" H 9000 4740 20  0001 C CNN
-F 1 "+5V" H 9000 4740 30  0000 C CNN
-F 2 "" H 9000 4650 60  0000 C CNN
-F 3 "" H 9000 4650 60  0000 C CNN
-	1    9000 4650
+P 9050 5100
+F 0 "#PWR032" H 9050 5190 20  0001 C CNN
+F 1 "+5V" H 9050 5190 30  0000 C CNN
+F 2 "" H 9050 5100 60  0000 C CNN
+F 3 "" H 9050 5100 60  0000 C CNN
+	1    9050 5100
 	1    0    0    -1
 $EndComp
@@
 L GND #PWR034
 U 1 1 54D2DCBF
-P 6050 5000
-F 0 "#PWR034" H 6050 5000 30  0001 C CNN
-F 1 "GND" H 6050 4930 30  0001 C CNN
-F 2 "" H 6050 5000 60  0000 C CNN
-F 3 "" H 6050 5000 60  0000 C CNN
-	1    6050 5000
+P 5900 4950
+F 0 "#PWR034" H 5900 4950 30  0001 C CNN
+F 1 "GND" H 5900 4880 30  0001 C CNN
+F 2 "" H 5900 4950 60  0000 C CNN
+F 3 "" H 5900 4950 60  0000 C CNN
+	1    5900 4950
 	1    0    0    -1
 $EndComp
@@
 L GND #PWR037
 U 1 1 54D2DCEC
-P 4900 2950
-F 0 "#PWR037" H 4900 2950 30  0001 C CNN
-F 1 "GND" H 4900 2880 30  0001 C CNN
-F 2 "" H 4900 2950 60  0000 C CNN
-F 3 "" H 4900 2950 60  0000 C CNN
-	1    4900 2950
+P 4900 2800
+F 0 "#PWR037" H 4900 2800 30  0001 C CNN
+F 1 "GND" H 4900 2730 30  0001 C CNN
+F 2 "" H 4900 2800 60  0000 C CNN
+F 3 "" H 4900 2800 60  0000 C CNN
+	1    4900 2800
 	1    0    0    -1
 $EndComp
 Wire Wire Line
-	4900 2800 4900 2950
+	4900 2600 4900 2800
 Wire Wire Line
-	4200 1900 4200 1700
+	4050 1700 4200 1700
 Wire Wire Line
-	5250 1350 4900 1400
+	5050 1200 4900 1200
 Wire Wire Line
 	4250 3400 4100 3400
@@
 	2200 3400 2400 3400
 Wire Wire Line
-	1300 3850 1300 3900
-Wire Wire Line
-	1300 3900 1500 4300
+	1300 4300 1500 4300
 Wire Wire Line
 	2200 4800 2200 4950
@@
 	4100 4800 4100 4950
 Wire Wire Line
-	5900 4800 6050 5000
+	5900 4800 5900 4950
 Wire Wire Line
-	9000 4650 9000 4700
-Wire Wire Line
-	9000 4700 8850 5100
+	9050 5100 8850 5100
 Wire Wire Line
 	8150 5600 8150 5750
 Wire Wire Line
 	7150 4700 7400 4700
-Text GLabel 5250 1350 2    60   Input ~ 0
+Text GLabel 5050 1200 2    60   Input ~ 0
 S1 Bus
 $Comp
 L FBR211 U26
 U 1 1 54D2DC25
-P 4900 2100
-F 0 "U26" H 5250 1600 60  0000 C CNN
-F 1 "inv5c" H 4900 2100 60  0000 C CNN
-F 2 "~" H 3900 2050 60  0000 C CNN
-F 3 "~" H 3900 2050 60  0000 C CNN
-	1    4900 2100
+P 4900 1900
+F 0 "U26" H 5250 1400 60  0000 C CNN
+F 1 "inv5c" H 4900 1900 60  0000 C CNN
+F 2 "~" H 3900 1850 60  0000 C CNN
+F 3 "~" H 3900 1850 60  0000 C CNN
+	1    4900 1900
 	-1   0    0    -1
 $EndComp

Commit message: more updates
Parts:
- U24, U25, U26, U27, U28: footprint ~ -> custom:211ARelay
Changed lines of the file:
@@
 F 0 "U24" H 2550 3600 60  0000 C CNN
 F 1 "and5a" H 2200 4100 60  0000 C CNN
-F 2 "~" H 1200 4050 60  0000 C CNN
+F 2 "custom:211ARelay" H 1200 4050 60  0000 C CNN
 F 3 "~" H 1200 4050 60  0000 C CNN
 	1    2200 4100
@@
 F 0 "U25" H 4450 3600 60  0000 C CNN
 F 1 "and5b" H 4100 4100 60  0000 C CNN
-F 2 "~" H 3100 4050 60  0000 C CNN
+F 2 "custom:211ARelay" H 3100 4050 60  0000 C CNN
 F 3 "~" H 3100 4050 60  0000 C CNN
 	1    4100 4100
@@
 F 0 "U27" H 6250 3600 60  0000 C CNN
 F 1 "and5c" H 5900 4100 60  0000 C CNN
-F 2 "~" H 4900 4050 60  0000 C CNN
+F 2 "custom:211ARelay" H 4900 4050 60  0000 C CNN
 F 3 "~" H 4900 4050 60  0000 C CNN
 	1    5900 4100
@@
 F 0 "U28" H 8500 4400 60  0000 C CNN
 F 1 "or3c" H 8150 4900 60  0000 C CNN
-F 2 "~" H 7150 4850 60  0000 C CNN
+F 2 "custom:211ARelay" H 7150 4850 60  0000 C CNN
 F 3 "~" H 7150 4850 60  0000 C CNN
 	1    8150 4900
@@
 F 0 "U26" H 5250 1400 60  0000 C CNN
 F 1 "inv5c" H 4900 1900 60  0000 C CNN
-F 2 "~" H 3900 1850 60  0000 C CNN
+F 2 "custom:211ARelay" H 3900 1850 60  0000 C CNN
 F 3 "~" H 3900 1850 60  0000 C CNN
 	1    4900 1900
