File: ALU/kicad/1BitALU/sectionE.sch (KiCad schematic (older format))
At the start: 6 parts, among them U29 and6a, U30 inv6b, U31 and6b, U32 inv6c, U33 and6c, U34 or3d

Commit message: * improvements
Connections:
- net +5V: now also U32.1 (IN); no longer U32.12 (IN)
Other:
- moved on the sheet: U29, U30, U31, U32, U33, U34

Commit message: more updates
Parts:
- U29, U30, U31, U32, U33, U34: footprint ~ -> custom:211ARelay
Changed lines of the file:
@@
 F 0 "U29" H 3150 3750 60  0000 C CNN
 F 1 "and6a" H 2800 4250 60  0000 C CNN
-F 2 "~" H 1800 4200 60  0000 C CNN
+F 2 "custom:211ARelay" H 1800 4200 60  0000 C CNN
 F 3 "~" H 1800 4200 60  0000 C CNN
 	1    2800 4250
@@
 F 0 "U31" H 4950 3750 60  0000 C CNN
 F 1 "and6b" H 4600 4250 60  0000 C CNN
-F 2 "~" H 3600 4200 60  0000 C CNN
+F 2 "custom:211ARelay" H 3600 4200 60  0000 C CNN
 F 3 "~" H 3600 4200 60  0000 C CNN
 	1    4600 4250
@@
 F 0 "U33" H 6700 3750 60  0000 C CNN
 F 1 "and6c" H 6350 4250 60  0000 C CNN
-F 2 "~" H 5350 4200 60  0000 C CNN
+F 2 "custom:211ARelay" H 5350 4200 60  0000 C CNN
 F 3 "~" H 5350 4200 60  0000 C CNN
 	1    6350 4250
@@
 F 0 "U34" H 8750 4250 60  0000 C CNN
 F 1 "or3d" H 8400 4750 60  0000 C CNN
-F 2 "~" H 7400 4700 60  0000 C CNN
+F 2 "custom:211ARelay" H 7400 4700 60  0000 C CNN
 F 3 "~" H 7400 4700 60  0000 C CNN
 	1    8400 4750
@@
 F 0 "U32" H 5950 1950 60  0000 C CNN
 F 1 "inv6c" H 5600 2450 60  0000 C CNN
-F 2 "~" H 4600 2400 60  0000 C CNN
+F 2 "custom:211ARelay" H 4600 2400 60  0000 C CNN
 F 3 "~" H 4600 2400 60  0000 C CNN
 	1    5600 2450
@@
 F 0 "U30" H 4200 1950 60  0000 C CNN
 F 1 "inv6b" H 3850 2450 60  0000 C CNN
-F 2 "~" H 2850 2400 60  0000 C CNN
+F 2 "custom:211ARelay" H 2850 2400 60  0000 C CNN
 F 3 "~" H 2850 2400 60  0000 C CNN
 	1    3850 2450
