File: ALU/kicad/1BitALU/1BitALU.kicad_pcb (KiCad board)
At the start: 2 copper layers, 165.1 x 165.1 mm, 55 parts, among them P1 CONN_6, P2 CONN_2, P3 Power, U1 xor3a, U10 and3a, U11 or2a, U12 and3b, U13 inv3b, U14 and3c, U15 or3a, U16 xor1b, U17 xor1a, U18 xor2b, U19 and4a, U2 and2a, U20 xor2a, U21 and4b, U22 and4c, U23 or3b, U24 and5a, U25 and5b, U26 inv5c, U27 and5c, U28 or3c, U29 and6a, U3 xor3b, U30 inv6b, U31 and6b, U32 inv6c, U33 and6c, U34 or3d, U4 and2b, U5 or1b, U6 and1a, U7 and1b, U8 or1a, U9 or2b

Commit message: * improvements
Parts:
- moved U32 14.6 mm to (156.8, 134.6), turned to 270 degrees
- moved R9 10.8 mm to (165.1, 156.8)
- moved P3 9.44 mm to (172.1, 168.3)
- moved D9 9.03 mm to (172.1, 158.1)
- moved U24 7.24 mm to (131.4, 88.9)
- moved U25 7.24 mm to (131.4, 104.1)
- moved U27 7.24 mm to (131.4, 119.4)
- moved U29 7.24 mm to (156.8, 73.7)
- moved U30 7.24 mm to (156.8, 104.1)
- moved U31 7.24 mm to (156.8, 88.9)
- moved U33 7.24 mm to (156.8, 119.4)
- moved U28 7.24 mm to (131.4, 149.9)
- moved U34 7.24 mm to (156.8, 149.9)
- moved U16 7.24 mm to (103.5, 43.2)
- moved U17 7.24 mm to (95.9, 71.1)
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Connections:
- U1 pad 1: (no net) -> Net-(U1-Pad1)
- U10 pad 1: (no net) -> Net-(U10-Pad1)
- U10 pad 7: (no net) -> Net-(U10-Pad7)
- U11 pad 1: (no net) -> Net-(U11-Pad1)
- U11 pad 7: (no net) -> Net-(U11-Pad7)
- U12 pad 12: (no net) -> Net-(U12-Pad12)
- U12 pad 7: (no net) -> Net-(U12-Pad7)
- U13 pad 1: (no net) -> Net-(U13-Pad1)
- U13 pad 6: (no net) -> Net-(U13-Pad6)
- U14 pad 12: (no net) -> Net-(U14-Pad12)
- U14 pad 7: (no net) -> Net-(U14-Pad7)
- U15 pad 1: (no net) -> Net-(U15-Pad1)
- U15 pad 7: (no net) -> Net-(U15-Pad7)
- U16 pad 1: (no net) -> Net-(U16-Pad1)
- U17 pad 1: (no net) -> Net-(U17-Pad1)
- U18 pad 1: (no net) -> Net-(U18-Pad1)
- U19 pad 1: (no net) -> Net-(U19-Pad1)
- U19 pad 7: (no net) -> Net-(U19-Pad7)
- U2 pad 12: (no net) -> Net-(U2-Pad12)
- U2 pad 7: (no net) -> Net-(U2-Pad7)
- U20 pad 12: (no net) -> Net-(U20-Pad12)
- U21 pad 12: (no net) -> Net-(U21-Pad12)
- U21 pad 7: (no net) -> Net-(U21-Pad7)
- U22 pad 12: (no net) -> Net-(U22-Pad12)
- U22 pad 7: (no net) -> Net-(U22-Pad7)
- U23 pad 1: (no net) -> Net-(U23-Pad1)
- U23 pad 7: (no net) -> Net-(U23-Pad7)
- U24 pad 1: (no net) -> Net-(U24-Pad1)
- U24 pad 7: (no net) -> Net-(U24-Pad7)
- U25 pad 12: (no net) -> Net-(U25-Pad12)
- U25 pad 7: (no net) -> Net-(U25-Pad7)
- U26 pad 12: (no net) -> Net-(U26-Pad12)
- U26 pad 6: (no net) -> Net-(U26-Pad6)
- U27 pad 12: (no net) -> Net-(U27-Pad12)
- U27 pad 7: (no net) -> Net-(U27-Pad7)
- U28 pad 1: (no net) -> Net-(U28-Pad1)
- U28 pad 7: (no net) -> Net-(U28-Pad7)
- U29 pad 12: (no net) -> Net-(U29-Pad12)
- U29 pad 7: (no net) -> Net-(U29-Pad7)
- U3 pad 12: (no net) -> Net-(U3-Pad12)
- U30 pad 12: (no net) -> Net-(U30-Pad12)
- U30 pad 6: (no net) -> Net-(U30-Pad6)
- U31 pad 12: (no net) -> Net-(U31-Pad12)
- U31 pad 7: (no net) -> Net-(U31-Pad7)
- U32 pad 1: (no net) -> +5V
- U32 pad 12: +5V -> Net-(U32-Pad12)
- U32 pad 6: (no net) -> Net-(U32-Pad6)
- U33 pad 12: (no net) -> Net-(U33-Pad12)
- U33 pad 7: (no net) -> Net-(U33-Pad7)
- U34 pad 12: (no net) -> Net-(U34-Pad12)
- U34 pad 7: (no net) -> Net-(U34-Pad7)
- U4 pad 1: (no net) -> Net-(U4-Pad1)
- U4 pad 7: (no net) -> Net-(U4-Pad7)
- U5 pad 1: (no net) -> Net-(U5-Pad1)
- U5 pad 7: (no net) -> Net-(U5-Pad7)
- U6 pad 1: (no net) -> Net-(U6-Pad1)
- U6 pad 7: (no net) -> Net-(U6-Pad7)
- U7 pad 12: (no net) -> Net-(U7-Pad12)
- U7 pad 7: (no net) -> Net-(U7-Pad7)
- U8 pad 1: (no net) -> Net-(U8-Pad1)
- U8 pad 7: (no net) -> Net-(U8-Pad7)
- U9 pad 1: (no net) -> Net-(U9-Pad1)
- U9 pad 7: (no net) -> Net-(U9-Pad7)
Routing:
- net GND: track 1040.1 -> 983.4 mm, vias 24 -> 22
- net +5V: track 653.4 -> 619.5 mm
- net S1 Bus: track 591.8 -> 562.6 mm
- net B Actual: track 144.1 -> 121.3 mm
- net Net-(U32-Pad7): track 10.2 -> 25.4 mm
- net XOR Out: track 116.8 -> 102.2 mm, vias 4 -> 5
- net AND Out: track 93.3 -> 80.0 mm
- net Cout: track 290.8 -> 281.9 mm
- net Net-(U25-Pad6): track 2.54 -> 7.62 mm
- net Net-(U21-Pad6): track 2.54 -> 7.62 mm
- net Net-(U16-Pad7): track 2.54 -> 7.62 mm
- net Net-(U16-Pad6): track 2.54 -> 7.62 mm
- net Cin: track 383.2 -> 378.5 mm
- net ADD Out: track 53.6 -> 49.3 mm
- net A: track 353.1 -> 349.0 mm
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Other:
- board size 165.1 x 165.1 mm -> 158.8 x 158.8 mm

Commit message: more updates
Parts:
- D1, D2, D3, D4, D5, D6, D7, D8, D9: footprint LED-3MM -> custom:90LED
- P1: footprint PIN_ARRAY-6X1 -> Socket_Strips:Socket_Strip_Angled_1x06
- P2, P3: footprint PIN_ARRAY_2X1 -> Socket_Strips:Socket_Strip_Angled_1x02
- R1, R2, R3, R4, R5, R6, R7, R8, R9: footprint R4 -> Discret:R4
- U1, U10, U11, U12, U13, U14, U15, U16, U17, U18, U19, U2, U20, U21, U22, U23, U24, U25, U26, U27, U28, U29, U3, U30, U31, U32, U33, U34, U4, U5, U6, U7, U8, U9: footprint 211ARelay -> custom:211ARelay
- moved D9 11.4 mm to (171.4, 146.7), turned to 0 degrees
- moved P1 9.03 mm to (165.1, 29.8), turned to 90 degrees
- moved P2 7.01 mm to (165.1, 37.5), turned to 90 degrees
- moved P3 6.48 mm to (165.7, 169.5), turned to 90 degrees
- moved D1 5.12 mm to (171.4, 41.9), turned to 0 degrees
- moved D2 5.12 mm to (171.4, 48.3), turned to 0 degrees
- moved D4 5.12 mm to (171.4, 61.0), turned to 0 degrees
- moved D3 5.12 mm to (171.4, 54.6), turned to 0 degrees
- moved D5 5.12 mm to (171.4, 67.3), turned to 0 degrees
- moved D6 5.12 mm to (171.4, 73.7), turned to 0 degrees
- moved D7 5.12 mm to (171.4, 80.0), turned to 0 degrees
- moved D8 5.12 mm to (171.4, 86.4), turned to 0 degrees
Routing:
- net Cin: track 378.5 -> 283.2 mm, vias 5 -> 6
- net GND: track 983.4 -> 1060.7 mm, vias 22 -> 24
- net Cout: track 281.9 -> 220.9 mm
- net S1 Bus: track 562.6 -> 537.8 mm, vias 5 -> 4
- net S0 Bus: track 584.2 -> 605.2 mm
- net OUT: track 363.1 -> 382.8 mm
- net B: track 180.3 -> 189.9 mm
- net Binv: track 186.7 -> 178.4 mm
- net A: track 349.0 -> 354.8 mm, vias 6 -> 7
- net +5V: track 619.5 -> 625.2 mm, vias 14 -> 15
- net Net-(U25-Pad6): track 7.62 -> 2.54 mm
- net Net-(U21-Pad6): track 7.62 -> 2.54 mm
- net Net-(U16-Pad7): track 7.62 -> 2.54 mm
- net Net-(U16-Pad6): track 7.62 -> 2.54 mm
- net Net-(D8-Pad1): track 35.9 -> 31.7 mm
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
Commit message: interim version
Parts:
- moved U9 120.8 mm to (166.7, 47.9), turned to 180 degrees
- moved P1 118.5 mm to (195.3, 144.5), turned to 0 degrees
- moved U3 114.2 mm to (181.9, 65.1), turned to 180 degrees
- moved P3 113.0 mm to (56.2, 141.9), turned to 270 degrees
- moved D1 109.5 mm to (183.2, 150.8), turned to 270 degrees
- moved P2 109.3 mm to (187.6, 144.5), turned to 0 degrees
- moved U11 108.2 mm to (151.4, 47.9), turned to 180 degrees
- moved U15 105.9 mm to (75.2, 47.9), turned to 180 degrees
- moved U7 105.1 mm to (62.5, 57.5), turned to 0 degrees
- moved D2 102.7 mm to (176.8, 150.8), turned to 270 degrees
- moved U10 98.7 mm to (136.2, 47.9), turned to 180 degrees
- moved U14 97.3 mm to (90.5, 47.9), turned to 180 degrees
- moved D3 96.2 mm to (170.5, 150.8), turned to 270 degrees
- moved U12 93.4 mm to (121.0, 47.9), turned to 180 degrees
- moved D9 93.1 mm to (78.4, 150.8), turned to 270 degrees
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Routing:
- net S0 Bus: track 605.2 -> 429.4 mm, vias 5 -> 6
- net GND: track 1060.7 -> 890.6 mm, vias 24 -> 25
- net +5V: track 625.2 -> 570.5 mm, vias 15 -> 11
- net S1 Bus: track 537.8 -> 494.0 mm
- net OUT: track 382.8 -> 349.6 mm, vias 7 -> 3
- net A: track 354.8 -> 324.5 mm, vias 7 -> 6
- net Binv: track 178.4 -> 154.9 mm
- net Cin: track 283.2 -> 296.7 mm, vias 6 -> 5
- net Cout: track 220.9 -> 208.3 mm, vias 4 -> 3
- net B: track 189.9 -> 177.8 mm
- net B Actual: track 121.3 -> 110.2 mm
- net ADD Out: track 49.3 -> 38.3 mm
- net AND Out: track 80.0 -> 70.4 mm
- net XOR Out: track 105.4 -> 95.9 mm
- net Net-(D9-Pad1): track 6.35 -> 12.1 mm
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Other:
- board size 158.8 x 158.8 mm -> 171.5 x 127 mm
- net class Power: clearance 0.635 -> 0.508; trace_width 1.27 -> 1.016

Commit message: interim version
Routing:
- net S1 Bus: track 494.0 -> 490.2 mm
- net +5V: track 570.5 -> 567.1 mm
Changed lines of the file:
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@@
     (thickness 1.6)
     (drawings 22)
-    (tracks 439)
+    (tracks 436)
     (zones 0)
     (modules 55)
@@
     (effects (font (size 1.5 1.5) (thickness 0.3)))
   )
-  (gr_text Power (at 66.9925 148.2725) (layer F.SilkS)
+  (gr_text Power (at 49.8475 138.7475) (layer F.SilkS)
     (effects (font (size 1.5 1.5) (thickness 0.3)))
   )
@@
   (via (at 50.4825 151.4475) (size 4.318) (drill 4.064) (layers F.Cu B.Cu) (net 0))
   (via (at 50.4825 35.8775) (size 4.318) (drill 4.064) (layers F.Cu B.Cu) (net 0))
-  (segment (start 55.5625 124.1425) (end 55.5625 141.2875) (width 1.016) (layer F.Cu) (net 1) (status 800000))
-  (segment (start 55.5625 141.2875) (end 56.1975 141.9225) (width 1.016) (layer F.Cu) (net 1) (status C00000))
-  (segment (start 75.2475 124.1425) (end 55.5625 124.1425) (width 1.016) (layer F.Cu) (net 1))
-  (segment (start 55.5625 98.7425) (end 55.5625 124.7775) (width 1.016) (layer F.Cu) (net 1))
-  (segment (start 55.5625 124.7775) (end 55.5625 124.1425) (width 1.016) (layer F.Cu) (net 1))
+  (segment (start 56.1975 98.7425) (end 56.1975 53.0225) (width 1.016) (layer F.Cu) (net 1))
+  (segment (start 56.1975 124.1425) (end 56.1975 98.7425) (width 1.016) (layer F.Cu) (net 1))
+  (segment (start 56.1975 141.9225) (end 56.1975 124.1425) (width 1.016) (layer F.Cu) (net 1) (status 400000))
+  (segment (start 75.2475 114.6175) (end 77.7875 114.6175) (width 1.016) (layer B.Cu) (net 1) (status C00000))
+  (segment (start 75.2475 124.1425) (end 56.1975 124.1425) (width 1.016) (layer F.Cu) (net 1))
   (segment (start 89.8525 145.0975) (end 100.0125 145.0975) (width 0.508) (layer B.Cu) (net 1))
   (via (at 100.0125 124.1425) (size 1.4224) (layers F.Cu B.Cu) (net 1))
@@
   (segment (start 136.2075 47.9425) (end 136.2075 53.0225) (width 1.016) (layer B.Cu) (net 1))
   (via (at 136.2075 53.0225) (size 1.4224) (layers F.Cu B.Cu) (net 1))
-  (segment (start 55.5625 53.0225) (end 75.2475 53.0225) (width 1.016) (layer F.Cu) (net 1))
+  (segment (start 56.1975 53.0225) (end 75.2475 53.0225) (width 1.016) (layer F.Cu) (net 1))
   (segment (start 75.2475 53.0225) (end 77.7875 53.0225) (width 1.016) (layer F.Cu) (net 1))
   (segment (start 77.7875 53.0225) (end 93.0275 53.0225) (width 1.016) (layer F.Cu) (net 1))
@@
   (segment (start 136.2075 53.0225) (end 151.4475 53.0225) (width 1.016) (layer F.Cu) (net 1))
   (segment (start 151.4475 53.0225) (end 166.6875 53.0225) (width 1.016) (layer F.Cu) (net 1))
-  (segment (start 55.5625 53.0225) (end 55.5625 98.7425) (width 1.016) (layer F.Cu) (net 1))
   (segment (start 166.6875 53.0225) (end 166.6875 47.9425) (width 1.016) (layer F.Cu) (net 1) (status 20))
   (segment (start 75.2475 92.3925) (end 75.2475 98.7425) (width 1.016) (layer F.Cu) (net 1))
   (segment (start 108.2675 98.7425) (end 75.2475 98.7425) (width 1.016) (layer F.Cu) (net 1))
-  (segment (start 75.2475 98.7425) (end 55.5625 98.7425) (width 1.016) (layer F.Cu) (net 1))
+  (segment (start 75.2475 98.7425) (end 56.1975 98.7425) (width 1.016) (layer F.Cu) (net 1))
   (via (at 151.4475 124.1425) (size 1.4224) (layers F.Cu B.Cu) (net 1))
   (segment (start 136.2075 124.1425) (end 120.9675 124.1425) (width 1.016) (layer F.Cu) (net 1))
@@
   (segment (start 120.9675 124.1425) (end 100.0125 124.1425) (width 1.016) (layer F.Cu) (net 1))
   (segment (start 100.0125 124.1425) (end 90.4875 124.1425) (width 1.016) (layer F.Cu) (net 1))
-  (segment (start 77.7875 114.6175) (end 75.2475 114.6175) (width 1.27) (layer B.Cu) (net 1) (status 30))
   (segment (start 151.4475 98.7425) (end 108.2675 98.7425) (width 1.016) (layer F.Cu) (net 1))
   (segment (start 90.4875 128.5875) (end 90.4875 124.1425) (width 1.016) (layer F.Cu) (net 1) (status 10))
@@
   (segment (start 87.9475 120.9675) (end 80.3275 128.5875) (width 0.635) (layer B.Cu) (net 14) (status 20))
   (segment (start 87.9475 118.4275) (end 87.9475 120.9675) (width 0.635) (layer B.Cu) (net 14))
-  (segment (start 87.9475 114.6175) (end 87.9475 118.4275) (width 0.635) (layer B.Cu) (net 14) (status 10))
   (segment (start 80.3275 84.7725) (end 80.3275 78.4225) (width 0.635) (layer F.Cu) (net 14) (status 10))
   (via (at 87.9475 118.4275) (size 1.4224) (layers F.Cu B.Cu) (net 14))

Commit message: interim version
Parts:
- moved P3 7.01 mm to (63.2, 142.6)
Routing:
- net (no net): track 0.00 -> 24.0 mm
- net +5V: track 567.1 -> 574.7 mm, vias 11 -> 12
- net GND: track 890.6 -> 894.1 mm
Other:
- board size 171.5 x 127 mm -> 165.1 x 120.7 mm
Changed lines of the file:
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@@
     (thickness 1.6)
     (drawings 22)
-    (tracks 436)
+    (tracks 443)
     (zones 0)
     (modules 55)
@@
   )
   (module Socket_Strips:Socket_Strip_Angled_1x02 (layer F.Cu)
-    (at 56.1975 141.9225 270)
+    (at 63.1825 142.5575 270)
     (descr "Through hole socket strip")
     (tags "socket strip")
@@
       (net 109 "Net-(U33-Pad6)"))
   )
-  (gr_line (start 217.4494 155.9052) (end 217.4494 28.9052) (angle 90) (layer Edge.Cuts) (width 0.15))
-  (gr_line (start 46.0375 31.4325) (end 217.4875 31.4325) (angle 90) (layer Edge.Cuts) (width 0.15))
-  (gr_line (start 45.9994 155.9052) (end 45.9994 28.9052) (angle 90) (layer Edge.Cuts) (width 0.15))
-  (gr_line (start 217.4494 155.9052) (end 45.9994 155.9052) (angle 90) (layer Edge.Cuts) (width 0.15))
+  (gr_line (start 52.3875 155.8925) (end 217.4875 155.8925) (angle 90) (layer Edge.Cuts) (width 0.15))
+  (gr_line (start 52.3875 35.2425) (end 52.3875 155.8925) (angle 90) (layer Edge.Cuts) (width 0.15))
+  (gr_line (start 217.4875 35.2425) (end 52.3875 35.2425) (angle 90) (layer Edge.Cuts) (width 0.15))
+  (gr_line (start 217.4875 155.8925) (end 217.4875 35.2425) (angle 90) (layer Edge.Cuts) (width 0.15))
   (gr_text Binv (at 166.6875 144.4625) (layer F.SilkS)
     (effects (font (size 1.5 1.5) (thickness 0.3)))
   )
-  (gr_text "1 Bit Relay Based ALU - Designed in Philadelphia by Vincent E. Fumo" (at 132.3975 35.2425) (layer F.SilkS)
+  (gr_text "1 Bit Relay Based ALU - Designed in Philadelphia by Vincent E. Fumo" (at 110.8075 37.1475) (layer F.SilkS)
     (effects (font (size 1.5 1.5) (thickness 0.3)))
   )
-  (gr_text Power (at 49.8475 138.7475) (layer F.SilkS)
+  (gr_text Power (at 56.1975 138.1125) (layer F.SilkS)
     (effects (font (size 1.5 1.5) (thickness 0.3)))
   )
@@
     (effects (font (size 1.5 1.5) (thickness 0.3)))
   )
+  (segment (start 153.3525 110.1725) (end 159.0675 110.1725) (width 1.016) (layer F.Cu) (net 0))
+  (segment (start 146.3675 108.2675) (end 150.8125 112.7125) (width 1.016) (layer F.Cu) (net 0))
+  (segment (start 155.2575 108.2675) (end 160.9725 108.2675) (width 1.016) (layer F.Cu) (net 0))
+  (segment (start 150.8125 112.7125) (end 153.3525 110.1725) (width 1.016) (layer F.Cu) (net 0))
+  (segment (start 153.3525 110.1725) (end 155.2575 108.2675) (width 1.016) (layer F.Cu) (net 0))
   (via (at 213.0044 151.4602) (size 4.318) (drill 4.064) (layers F.Cu B.Cu) (net 0))
-  (via (at 213.0425 35.8775) (size 4.318) (drill 4.064) (layers F.Cu B.Cu) (net 0))
-  (via (at 50.4825 151.4475) (size 4.318) (drill 4.064) (layers F.Cu B.Cu) (net 0))
-  (via (at 50.4825 35.8775) (size 4.318) (drill 4.064) (layers F.Cu B.Cu) (net 0))
+  (via (at 213.0425 39.6875) (size 4.318) (drill 4.064) (layers F.Cu B.Cu) (net 0))
+  (via (at 56.8325 151.4475) (size 4.318) (drill 4.064) (layers F.Cu B.Cu) (net 0))
+  (via (at 56.8325 39.6875) (size 4.318) (drill 4.064) (layers F.Cu B.Cu) (net 0))
+  (via (at 56.1975 124.1425) (size 1.4224) (layers F.Cu B.Cu) (net 1))
+  (segment (start 63.1825 142.5575) (end 56.1975 142.5575) (width 1.016) (layer B.Cu) (net 1) (status 400000))
+  (segment (start 56.1975 142.5575) (end 56.1975 124.1425) (width 1.016) (layer B.Cu) (net 1))
   (segment (start 56.1975 98.7425) (end 56.1975 53.0225) (width 1.016) (layer F.Cu) (net 1))
   (segment (start 56.1975 124.1425) (end 56.1975 98.7425) (width 1.016) (layer F.Cu) (net 1))
-  (segment (start 56.1975 141.9225) (end 56.1975 124.1425) (width 1.016) (layer F.Cu) (net 1) (status 400000))
-  (segment (start 75.2475 114.6175) (end 77.7875 114.6175) (width 1.016) (layer B.Cu) (net 1) (status C00000))
+  (segment (start 75.2475 114.6175) (end 77.7875 114.6175) (width 1.016) (layer B.Cu) (net 1))
   (segment (start 75.2475 124.1425) (end 56.1975 124.1425) (width 1.016) (layer F.Cu) (net 1))
   (segment (start 89.8525 145.0975) (end 100.0125 145.0975) (width 0.508) (layer B.Cu) (net 1))
@@
   (segment (start 105.7275 68.8975) (end 105.7275 66.3575) (width 0.635) (layer F.Cu) (net 9) (status 20))
   (segment (start 120.9675 70.8025) (end 105.7275 70.8025) (width 0.635) (layer F.Cu) (net 9))
-  (via (at 58.1025 135.5725) (size 1.4224) (layers F.Cu B.Cu) (net 10))
-  (segment (start 61.9125 139.3825) (end 58.1025 135.5725) (width 1.016) (layer F.Cu) (net 10))
-  (segment (start 61.9125 140.0175) (end 61.9125 139.3825) (width 1.016) (layer F.Cu) (net 10))
-  (segment (start 56.1975 144.4625) (end 61.9125 144.4625) (width 1.016) (layer F.Cu) (net 10))
-  (segment (start 61.9125 140.0175) (end 61.9125 144.4625) (width 1.016) (layer F.Cu) (net 10))
+  (segment (start 58.1025 121.6025) (end 58.1025 140.0175) (width 1.016) (layer B.Cu) (net 10))
+  (segment (start 58.1025 140.0175) (end 65.0875 140.0175) (width 1.016) (layer F.Cu) (net 10))
+  (via (at 58.1025 140.0175) (size 1.4224) (layers F.Cu B.Cu) (net 10))
+  (segment (start 63.1825 145.0975) (end 69.5325 145.0975) (width 1.016) (layer F.Cu) (net 10) (status 400000))
+  (segment (start 69.5325 145.0975) (end 69.5325 140.0175) (width 1.016) (layer F.Cu) (net 10))
   (segment (start 133.6675 57.4675) (end 133.6675 51.1175) (width 1.016) (layer B.Cu) (net 10))
   (via (at 133.6675 51.1175) (size 1.4224) (layers F.Cu B.Cu) (net 10))
@@
   (segment (start 136.2075 153.9875) (end 131.1275 153.9875) (width 0.508) (layer F.Cu) (net 10))
   (segment (start 131.1275 153.9875) (end 131.1275 140.0175) (width 0.508) (layer F.Cu) (net 10))
-  (segment (start 65.0875 140.0175) (end 61.9125 140.0175) (width 1.016) (layer F.Cu) (net 10))
   (segment (start 75.8825 150.8125) (end 75.8825 140.0175) (width 0.508) (layer F.Cu) (net 10) (status 10))
   (segment (start 58.1025 101.2825) (end 58.1025 74.6125) (width 1.016) (layer B.Cu) (net 10))
@@
   (segment (start 126.0475 101.2825) (end 141.2875 101.2825) (width 1.016) (layer F.Cu) (net 10))
   (segment (start 80.3275 140.0175) (end 75.8825 140.0175) (width 1.016) (layer F.Cu) (net 10))
-  (segment (start 75.8825 140.0175) (end 65.0875 140.0175) (width 1.016) (layer F.Cu) (net 10))
+  (segment (start 75.8825 140.0175) (end 69.5325 140.0175) (width 1.016) (layer F.Cu) (net 10))
+  (segment (start 69.5325 140.0175) (end 65.0875 140.0175) (width 1.016) (layer F.Cu) (net 10))
   (segment (start 95.5675 140.0175) (end 80.3275 140.0175) (width 1.016) (layer F.Cu) (net 10))
   (segment (start 110.8075 140.0175) (end 95.5675 140.0175) (width 1.016) (layer F.Cu) (net 10))
@@
   (via (at 58.1025 74.6125) (size 1.4224) (layers F.Cu B.Cu) (net 10))
   (segment (start 118.4275 74.6125) (end 58.1025 74.6125) (width 1.016) (layer F.Cu) (net 10))
-  (segment (start 58.1025 121.6025) (end 58.1025 135.5725) (width 1.016) (layer B.Cu) (net 10))
   (segment (start 138.7475 40.3225) (end 138.7475 44.7675) (width 0.508) (layer B.Cu) (net 11))
   (segment (start 126.0475 40.3225) (end 126.0475 44.7675) (width 0.508) (layer B.Cu) (net 11))
@@
   (segment (start 126.0475 44.7675) (end 138.7475 44.7675) (width 0.508) (layer B.Cu) (net 11))
   (segment (start 138.7475 44.7675) (end 153.9875 44.7675) (width 0.508) (layer B.Cu) (net 11))
-  (segment (start 62.5475 40.3225) (end 60.0075 40.3225) (width 1.016) (layer B.Cu) (net 12))
+  (segment (start 62.5475 40.3225) (end 62.5475 45.4025) (width 1.016) (layer B.Cu) (net 12) (status 400000))
+  (segment (start 62.5475 45.4025) (end 60.0075 45.4025) (width 1.016) (layer B.Cu) (net 12))
   (segment (start 207.9625 110.8075) (end 207.9625 144.4625) (width 1.016) (layer B.Cu) (net 12) (status 20))
   (segment (start 165.4175 110.8075) (end 207.9625 110.8075) (width 0.635) (layer F.Cu) (net 12))
@@
   (segment (start 62.5475 106.9975) (end 66.3575 103.1875) (width 1.016) (layer F.Cu) (net 12) (status 10))
   (segment (start 60.0075 104.4575) (end 60.0075 84.7725) (width 1.016) (layer B.Cu) (net 12))
-  (segment (start 60.0075 84.7725) (end 60.0075 40.3225) (width 1.016) (layer B.Cu) (net 12))
+  (segment (start 60.0075 84.7725) (end 60.0075 45.4025) (width 1.016) (layer B.Cu) (net 12))
   (segment (start 60.0075 106.9975) (end 60.0075 104.4575) (width 1.016) (layer B.Cu) (net 12))
   (segment (start 62.5475 106.9975) (end 60.0075 106.9975) (width 1.016) (layer B.Cu) (net 12) (status 10))
